File: KiCad/RCMhardwareByte.kicad_pcb (KiCad board)
At the start: 4 copper layers, 31.8 x 31.8 mm, 61 parts, among them IC1 TMC7300, IC2 TMC7300, IC3 TMC7300, IC4 TMC7300, J1 pads to solder wires to, reco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, J2 1x08 male header pins, J3 1x08 male header pins, J4 1x08 male header pins, J5 1x08 male header pins, J6 2x08 female header pins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

Commit message: v2.3.0
Parts:
- TP1: value TestPoint -> usb
- TP2: value TestPoint -> vbat
- TP3: value TestPoint -> 5V pwr
- TP4: value TestPoint -> gnd
Routing:
- net GND: vias 59 -> 60
Other:
- board text added: "5V"
- board text added: "V2.3"
- board text removed: "V2.2"
- board text removed: "esp"
