File: KiCad/RCMhardwareByte.kicad_sch (KiCad schematic)
At the start: 61 parts, among them IC1 TMC7300, IC2 TMC7300, IC3 TMC7300, IC4 TMC7300, J1 pads to solder wires to, reco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, J2 1x08 male header pins, J3 1x08 male header pins, J4 1x08 male header pins, J5 1x08 male header pins, J6 2x08 female header pins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

Commit message: v2.3.0
Parts:
- TP1: value TestPoint -> usb
- TP2: value TestPoint -> vbat
- TP3: value TestPoint -> 5V pwr
- TP4: value TestPoint -> gnd
Other:
- company: joshua-8 -> https://github.com/rcmgames/RCM-Hardware-BYTE
Changed lines of the file:
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@@
   (title_block
     (title "RCM Byte")
-    (rev "2.1")
-    (company "joshua-8")
+    (rev "2.3")
+    (company "https://github.com/rcmgames/RCM-Hardware-BYTE")
   )
   (junction (at 105.41 369.57) (diameter 0) (color 0 0 0 0)
@@
   )
   (symbol (lib_id "Connector:TestPoint") (at 346.71 251.46 0) (unit 1)
-    (in_bom yes) (on_board yes) (dnp no) (fields_autoplaced)
-    (property "Reference" "TP2" (at 349.25 246.888 0)
+    (in_bom yes) (on_board yes) (dnp no)
+    (property "Reference" "TP2" (at 346.71 246.38 0)
       (effects (font (size 1.27 1.27)) (justify left))
     )
-    (property "Value" "TestPoint" (at 349.25 249.428 0)
+    (property "Value" "vbat" (at 347.98 248.92 0)
       (effects (font (size 1.27 1.27)) (justify left))
     )
@@
   (symbol (lib_id "Connector:TestPoint") (at 337.82 262.89 180) (unit 1)
     (in_bom yes) (on_board yes) (dnp no)
-    (property "Reference" "TP4" (at 334.01 265.43 0)
+    (property "Reference" "TP4" (at 332.74 265.43 0)
       (effects (font (size 1.27 1.27)) (justify right))
     )
-    (property "Value" "TestPoint" (at 334.01 267.97 0)
+    (property "Value" "gnd" (at 334.01 267.97 0)
       (effects (font (size 1.27 1.27)) (justify right))
     )
@@
       (effects (font (size 1.27 1.27)) (justify left))
     )
-    (property "Value" "TestPoint" (at 447.04 36.83 0)
+    (property "Value" "5V pwr" (at 447.04 36.83 0)
       (effects (font (size 1.27 1.27)) (justify left))
     )
@@
       (effects (font (size 1.27 1.27)) (justify left))
     )
-    (property "Value" "TestPoint" (at 424.18 36.83 0)
+    (property "Value" "usb" (at 424.18 36.83 0)
       (effects (font (size 1.27 1.27)) (justify left))
     )
